File: M6/CPR Machine Schematic/MotorControl.kicad_sch (KiCad schematic)
At the start: 3 parts, among them U1 MCP2517FD CLICK, U3 Moteus-x1

Commit message: ToF
Connections:
- net at U1. (TXCAN): now also U3. (GND)
- new net: U1. (TXCAN), U3. (GND)

Commit message: morer kicad
Connections:
- net GND: no longer U1.8 (GND)
- net at U1. (TXCAN): now also U3. (GND)
- new net: U1. (TXCAN), U3. (GND)
- new net: U1.8 (GND), U3. (GND)
Changed lines of the file:
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@@
+	(wire
+		(pts
+			(xy 111.76 125.73) (xy 132.08 125.73)
+		)
+		(stroke
+			(width 0)
+			(type default)
+		)
+	)
+	(wire
+		(pts
+			(xy 111.76 91.44) (xy 111.76 125.73)
+		)
+		(stroke
+			(width 0)
+			(type default)
+		)
+	)
 	(wire
 		(pts
@@
 				(path "/8991fc77-975f-4978-a089-6b2a5e33f59b/5d577b9a-7e09-4b18-b019-9e51a9486569"
 					(reference "U1")
-					(unit 1)
-				)
-			)
-		)
-	)
-	(symbol
-		(lib_id "power:GND")
-		(at 132.08 125.73 0)
-		(unit 1)
-		(exclude_from_sim no)
-		(in_bom yes)
-		(on_board yes)
-		(dnp no)
-		(fields_autoplaced yes)
-		(property "Reference" "#PWR02"
-			(at 132.08 132.08 0)
-			(effects
-				(font
-					(size 1.27 1.27)
-				)
-				(hide yes)
-			)
-		)
-		(property "Value" "GND"
-			(at 132.08 130.81 0)
-			(effects
-				(font
-					(size 1.27 1.27)
-				)
-			)
-		)
-		(property "Footprint" ""
-			(at 132.08 125.73 0)
-			(effects
-				(font
-					(size 1.27 1.27)
-				)
-				(hide yes)
-			)
-		)
-		(property "Datasheet" ""
-			(at 132.08 125.73 0)
-			(effects
-				(font
-					(size 1.27 1.27)
-				)
-				(hide yes)
-			)
-		)
-		(property "Description" "Power symbol creates a global label with name \"GND\" , ground"
-			(at 132.08 125.73 0)
-			(effects
-				(font
-					(size 1.27 1.27)
-				)
-				(hide yes)
-			)
-		)
-		(pin "1"
-		)
-		(instances
-			(project ""
-				(path "/8991fc77-975f-4978-a089-6b2a5e33f59b/5d577b9a-7e09-4b18-b019-9e51a9486569"
-					(reference "#PWR02")
 					(unit 1)
 				)
@@
 					(unit 1)
 				)
-			)
-		)
-	)
-	(symbol
-		(lib_id "power:GND")
-		(at 111.76 91.44 0)
-		(unit 1)
-		(exclude_from_sim no)
-		(in_bom yes)
-		(on_board yes)
-		(dnp no)
-		(fields_autoplaced yes)
-		(property "Reference" "#PWR05"
-			(at 111.76 97.79 0)
-			(effects
-				(font
-					(size 1.27 1.27)
-				)
-				(hide yes)
-			)
-		)
-		(property "Value" "GND"
-			(at 111.76 96.52 0)
-			(effects
-				(font
-					(size 1.27 1.27)
-				)
-			)
-		)
-		(property "Footprint" ""
-			(at 111.76 91.44 0)
-			(effects
-				(font
-					(size 1.27 1.27)
-				)
-				(hide yes)
-			)
-		)
-		(property "Datasheet" ""
-			(at 111.76 91.44 0)
-			(effects
-				(font
-					(size 1.27 1.27)
-				)
-				(hide yes)
-			)
-		)
-		(property "Description" "Power symbol creates a global label with name \"GND\" , ground"
-			(at 111.76 91.44 0)
-			(effects
-				(font
-					(size 1.27 1.27)
-				)
-				(hide yes)
-			)
-		)
-		(pin "1"
-		)
-		(instances
-			(project ""
-				(path "/8991fc77-975f-4978-a089-6b2a5e33f59b/5d577b9a-7e09-4b18-b019-9e51a9486569"
-					(reference "#PWR05")
-					(unit 1)
-				)

Commit message: HMI schem for real for real
Connections:
- net at U1. (TXCAN): now also U3. (GND)
- net CS renamed SPI_CS
- net INT renamed SPI_INT
- net SCK renamed SPI_SCK
- net SDI renamed SPI_SDI
- net SDO renamed SPI_SDO
- new net: U1. (TXCAN), U3. (GND)
Changed lines of the file:
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@@
 		)
 	)
-	(hierarchical_label "INT"
+	(hierarchical_label "SPI_SDO"
+		(shape output)
+		(at 132.08 118.11 180)
+		(effects
+			(font
+				(size 1.27 1.27)
+			)
+			(justify right)
+		)
+	)
+	(hierarchical_label "SPI_CS"
+		(shape input)
+		(at 132.08 113.03 180)
+		(effects
+			(font
+				(size 1.27 1.27)
+			)
+			(justify right)
+		)
+	)
+	(hierarchical_label "SPI_SDI"
+		(shape input)
+		(at 132.08 120.65 180)
+		(effects
+			(font
+				(size 1.27 1.27)
+			)
+			(justify right)
+		)
+	)
+	(hierarchical_label "SPI_INT"
 		(shape output)
 		(at 152.4 110.49 0)
@@
 		)
 	)
-	(hierarchical_label "SDI"
-		(shape input)
-		(at 132.08 120.65 180)
-		(effects
-			(font
-				(size 1.27 1.27)
-			)
-			(justify right)
-		)
-	)
-	(hierarchical_label "SCK"
+	(hierarchical_label "SPI_SCK"
 		(shape input)
 		(at 132.08 115.57 180)
 		(effects
 			(font
-				(size 1.27 1.27)
-			)
-			(justify right)
-		)
-	)
-	(hierarchical_label "SDO"
-		(shape output)
-		(at 132.08 118.11 180)
-		(effects
-			(font
-				(size 1.27 1.27)
-			)
-			(justify right)
-		)
-	)
-	(hierarchical_label "CS"
-		(shape input)
-		(at 132.08 113.03 180)
-		(effects
-			(font
