File: M6/CPR Machine Schematic/HMI_Teensy.kicad_sch (KiCad schematic)
At the start: 11 parts, among them IC1 74HC125, SW5 LED Button, SW6 LED Button, SW7 Non-LED Button, U10 AdafruitRA8875, U11 MAX98357A, U9 AdafruitRA8875

Commit message: kicad saves
Other:
- moved on the sheet: R3, R4, SW5, SW6, SW7
