File: M6/CPR Machine Schematic/Microcontroller.kicad_sch (KiCad schematic)
At the start: 2 parts, among them U1 MCP2517FD CLICK, U2 Teensy4.1

Commit message: More Schematics
Parts:
- removed U1: MCP2517FD CLICK, symbol Custom_Parts:MCP2517FD_CLICK
Connections:
- net INT: now reaches U2.11 (9_OUT1C)
- net CS: now reaches U2.12 (10_CS_MQSR)
- net SDI: now reaches U2.13 (11_MOSI_CTX1)
- net SDO: now reaches U2.14 (12_MISO_MQSL)
- net SCK: now reaches U2.35 (13_SCK_LED)
- no-connect marks 4 -> 18
Other:
- moved on the sheet: U2

Commit message: ToF
Connections:
- net I2C_SDA: now reaches U2.40 (18_A4_SDA)
- net I2C_SCL: now reaches U2.41 (19_A5_SCL)
Changed lines of the file:
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@@
+		)
+	)
+	(hierarchical_label "I2C_SCL"
+		(shape output)
+		(at 170.18 71.12 0)
+		(effects
+			(font
+				(size 1.27 1.27)
+			)
+			(justify left)
+		)
+	)
+	(hierarchical_label "I2C_SDA"
+		(shape bidirectional)
+		(at 170.18 73.66 0)
+		(effects
+			(font
+				(size 1.27 1.27)
+			)
+			(justify left)
 		)
 	)

Commit message: morer kicad
Connections:
- net GND: now reaches U2.1 (GND)
- net GND: now also U2.34 (GND), U2.47 (GND)
- net UART_RX: now reaches U2.2 (0_RX1_CRX2_CS1)
- net UART_TX: now reaches U2.3 (1_TX1_CTX2_MISO1)
- net +5V: now reaches U2.48 (VIN)
- net CS renamed SPI_CS
- net INT renamed SPI_INT
- net SCK renamed SPI_SCK
- net SDI renamed SPI_SDI
- net SDO renamed SPI_SDO
- no-connect marks 18 -> 19

Commit message: HMI schem for real for real
Connections:
- net +3.3V: now reaches U2.46 (3V3)
- no-connect marks 19 -> 53
Changed lines of the file:
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@@
 	(paper "A4")
 	(no_connect
+		(at 114.3 106.68)
+	)
+	(no_connect
 		(at 142.24 140.97)
 	)
 	(no_connect
+		(at 114.3 68.58)
+	)
+	(no_connect
+		(at 114.3 93.98)
+	)
+	(no_connect
+		(at 114.3 66.04)
+	)
+	(no_connect
+		(at 114.3 63.5)
+	)
+	(no_connect
 		(at 114.3 133.35)
 	)
 	(no_connect
+		(at 114.3 96.52)
+	)
+	(no_connect
+		(at 170.18 99.06)
+	)
+	(no_connect
+		(at 114.3 76.2)
+	)
+	(no_connect
+		(at 170.18 109.22)
+	)
+	(no_connect
+		(at 170.18 81.28)
+	)
+	(no_connect
 		(at 114.3 130.81)
 	)
 	(no_connect
+		(at 170.18 106.68)
+	)
+	(no_connect
+		(at 170.18 66.04)
+	)
+	(no_connect
 		(at 138.43 140.97)
 	)
 	(no_connect
+		(at 114.3 109.22)
+	)
+	(no_connect
 		(at 114.3 128.27)
 	)
@@
 	)
 	(no_connect
+		(at 170.18 78.74)
+	)
+	(no_connect
 		(at 170.18 123.19)
 	)
 	(no_connect
+		(at 114.3 91.44)
+	)
+	(no_connect
+		(at 170.18 60.96)
+	)
+	(no_connect
+		(at 114.3 99.06)
+	)
+	(no_connect
 		(at 134.62 140.97)
 	)
 	(no_connect
+		(at 170.18 91.44)
+	)
+	(no_connect
+		(at 114.3 111.76)
+	)
+	(no_connect
+		(at 170.18 111.76)
+	)
+	(no_connect
 		(at 170.18 125.73)
 	)
@@
 	)
 	(no_connect
+		(at 170.18 93.98)
+	)
+	(no_connect
+		(at 170.18 68.58)
+	)
+	(no_connect
+		(at 114.3 88.9)
+	)
+	(no_connect
 		(at 170.18 128.27)
 	)
 	(no_connect
+		(at 114.3 60.96)
+	)
+	(no_connect
 		(at 114.3 123.19)
 	)
 	(no_connect
+		(at 170.18 63.5)
+	)
+	(no_connect
 		(at 114.3 119.38)
 	)
 	(no_connect
+		(at 170.18 104.14)
+	)
+	(no_connect
+		(at 170.18 101.6)
+	)
+	(no_connect
 		(at 146.05 140.97)
 	)
 	(no_connect
+		(at 114.3 73.66)
+	)
+	(no_connect
 		(at 170.18 120.65)
 	)
@@
 	)
 	(no_connect
+		(at 170.18 96.52)
+	)
+	(no_connect
+		(at 114.3 101.6)
+	)
+	(no_connect
 		(at 170.18 49.53)
 	)
 	(no_connect
+		(at 114.3 104.14)
+	)
+	(no_connect
+		(at 170.18 76.2)
+	)
+	(no_connect
 		(at 114.3 116.84)
 	)
 	(no_connect
+		(at 114.3 71.12)
+	)
+	(no_connect
 		(at 170.18 130.81)
+	)
+	(no_connect
+		(at 170.18 83.82)
 	)
 	(wire
@@
 	(wire
 		(pts
-			(xy 177.8 55.88) (xy 170.18 55.88)
+			(xy 181.61 55.88) (xy 170.18 55.88)
 		)
 		(stroke
@@
 	)
 	(symbol
+		(lib_id "power:+3.3V")
+		(at 170.18 58.42 270)
+		(unit 1)
+		(exclude_from_sim no)
+		(in_bom yes)
+		(on_board yes)
+		(dnp no)
+		(fields_autoplaced yes)
+		(property "Reference" "#PWR031"
+			(at 166.37 58.42 0)
+			(effects
+				(font
+					(size 1.27 1.27)
+				)
+				(hide yes)
+			)
+		)
+		(property "Value" "+3.3V"
+			(at 173.99 58.4199 90)
+			(effects
+				(font
+					(size 1.27 1.27)
+				)
+				(justify left)
+			)
+		)
+		(property "Footprint" ""
+			(at 170.18 58.42 0)
+			(effects
+				(font
+					(size 1.27 1.27)
+				)
+				(hide yes)
+			)
+		)
+		(property "Datasheet" ""
+			(at 170.18 58.42 0)
+			(effects
+				(font
+					(size 1.27 1.27)
+				)
+				(hide yes)
+			)
+		)
+		(property "Description" "Power symbol creates a global label with name \"+3.3V\""
+			(at 170.18 58.42 0)
+			(effects
+				(font
+					(size 1.27 1.27)
+				)
+				(hide yes)
+			)
+		)
+		(pin "1"
+		)
+		(instances
+			(project ""
+				(path "/8991fc77-975f-4978-a089-6b2a5e33f59b/8b2fecf3-fab6-4137-a5b1-aa5c7fdce798"
+					(reference "#PWR031")
+					(unit 1)
+				)
+			)
+		)
+	)
+	(symbol
 		(lib_id "power:+5V")
 		(at 170.18 53.34 270)
@@
 	(symbol
 		(lib_id "power:GND")
-		(at 177.8 55.88 0)
+		(at 181.61 55.88 0)
 		(unit 1)
 		(exclude_from_sim no)
@@
 		(fields_autoplaced yes)
 		(property "Reference" "#PWR022"
-			(at 177.8 62.23 0)
+			(at 181.61 62.23 0)
 			(effects
 				(font
@@
 		)
 		(property "Value" "GND"
-			(at 177.8 60.96 0)
+			(at 181.61 60.96 0)
 			(effects
 				(font
@@
 		)
 		(property "Footprint" ""
-			(at 177.8 55.88 0)
+			(at 181.61 55.88 0)
 			(effects
 				(font
@@
 		)
 		(property "Datasheet" ""
-			(at 177.8 55.88 0)
+			(at 181.61 55.88 0)
 			(effects
 				(font
@@
 		)
 		(property "Description" "Power symbol creates a global label with name \"GND\" , ground"
-			(at 177.8 55.88 0)
-			(effects
-				(font
+			(at 181.61 55.88 0)
+			(effects
+				(font

Commit message: Finalized kiCAD
Connections:
- net I2C_SCL: now also U2.37 (15_A1_RX3_SPDIF_IN); no longer U2.41 (19_A5_SCL)
- net I2C_SDA: now also U2.36 (14_A0_TX3_SPDIF_OUT); no longer U2.40 (18_A4_SDA)
- net White_Button: now reaches U2.17 (25_A11_RX6_SDA2)
- net Red_Button: now reaches U2.18 (26_A12_MOSI1)
- net Red_LED: now reaches U2.19 (27_A13_SCK1)
- net Green_Button: now reaches U2.20 (28_RX7)
- net Green_LED: now reaches U2.21 (29_TX7)
- net SPI_CS2: now reaches U2.38 (16_A2_RX4_SCL1)
- net SPI_CS3: now reaches U2.39 (17_A3_TX4_SDA1)
- net I2S_LRC: now reaches U2.42 (20_A6_TX5_LRCLK1)
- net I2S_BCLK: now reaches U2.43 (21_A7_RX5_BCLK1)
- net I2S_DIN: now reaches U2.44 (22_A8_CTX1)
- new net RST1: U2.41 (19_A5_SCL)
- new net RST2: U2.40 (18_A4_SDA)
- no-connect marks 53 -> 41
Changed lines of the file:
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@@
-	)
-	(no_connect
-		(at 114.3 93.98)
 	)
 	(no_connect
@@
 	)
 	(no_connect
-		(at 114.3 96.52)
-	)
-	(no_connect
 		(at 170.18 99.06)
 	)
@@
 	)
 	(no_connect
+		(at 170.18 60.96)
+	)
+	(no_connect
 		(at 170.18 109.22)
 	)
 	(no_connect
-		(at 170.18 81.28)
-	)
-	(no_connect
 		(at 114.3 130.81)
 	)
@@
 	)
 	(no_connect
-		(at 170.18 66.04)
-	)
-	(no_connect
 		(at 138.43 140.97)
 	)
@@
 	)
 	(no_connect
-		(at 170.18 78.74)
-	)
-	(no_connect
 		(at 170.18 123.19)
 	)
@@
 	)
 	(no_connect
-		(at 170.18 60.96)
-	)
-	(no_connect
-		(at 114.3 99.06)
-	)
-	(no_connect
 		(at 134.62 140.97)
 	)
@@
 	)
 	(no_connect
-		(at 170.18 68.58)
-	)
-	(no_connect
 		(at 114.3 88.9)
 	)
@@
 	)
 	(no_connect
-		(at 170.18 63.5)
-	)
-	(no_connect
 		(at 114.3 119.38)
 	)
@@
 	)
 	(no_connect
-		(at 114.3 101.6)
-	)
-	(no_connect
 		(at 170.18 49.53)
 	)
 	(no_connect
-		(at 114.3 104.14)
-	)
-	(no_connect
-		(at 170.18 76.2)
-	)
-	(no_connect
 		(at 114.3 116.84)
 	)
@@
 	(no_connect
 		(at 170.18 130.81)
-	)
-	(no_connect
-		(at 170.18 83.82)
 	)
 	(wire
@@
 		)
 	)
+	(hierarchical_label "SPI_CS3"
+		(shape output)
+		(at 170.18 76.2 0)
+		(effects
+			(font
+				(size 1.27 1.27)
+			)
+			(justify left)
+		)
+	)
 	(hierarchical_label "SPI_SDO"
 		(shape input)
@@
 		)
 	)
+	(hierarchical_label "Red_Button"
+		(shape output)
+		(at 114.3 96.52 180)
+		(effects
+			(font
+				(size 1.27 1.27)
+			)
+			(justify right)
+		)
+	)
+	(hierarchical_label "I2S_BCLK"
+		(shape output)
+		(at 170.18 66.04 0)
+		(effects
+			(font
+				(size 1.27 1.27)
+			)
+			(justify left)
+		)
+	)
+	(hierarchical_label "I2S_LRC"
+		(shape output)
+		(at 170.18 68.58 0)
+		(effects
+			(font
+				(size 1.27 1.27)
+			)
+			(justify left)
+		)
+	)
+	(hierarchical_label "RST1"
+		(shape output)
+		(at 170.18 71.12 0)
+		(effects
+			(font
+				(size 1.27 1.27)
+			)
+			(justify left)
+		)
+	)
+	(hierarchical_label "SPI_CS2"
+		(shape output)
+		(at 170.18 78.74 0)
+		(effects
+			(font
+				(size 1.27 1.27)
+			)
+			(justify left)
+		)
+	)
 	(hierarchical_label "SPI_SDI"
 		(shape output)
@@
 		)
 	)
+	(hierarchical_label "Green_Button"
+		(shape output)
+		(at 114.3 101.6 180)
+		(effects
+			(font
+				(size 1.27 1.27)
+			)
+			(justify right)
+		)
+	)
 	(hierarchical_label "I2C_SCL"
 		(shape output)
-		(at 170.18 71.12 0)
-		(effects
-			(font
-				(size 1.27 1.27)
-			)
-			(justify left)
+		(at 170.18 81.28 0)
+		(effects
+			(font
+				(size 1.27 1.27)
+			)
+			(justify left)
+		)
+	)
+	(hierarchical_label "Red_LED"
+		(shape output)
+		(at 114.3 99.06 180)
+		(effects
+			(font
+				(size 1.27 1.27)
+			)
+			(justify right)
 		)
 	)
@@
 	(hierarchical_label "I2C_SDA"
 		(shape bidirectional)
+		(at 170.18 83.82 0)
+		(effects
+			(font
+				(size 1.27 1.27)
+			)
+			(justify left)
+		)
+	)
+	(hierarchical_label "White_Button"
+		(shape output)
+		(at 114.3 93.98 180)
+		(effects
+			(font
+				(size 1.27 1.27)
+			)
+			(justify right)
+		)
+	)
+	(hierarchical_label "RST2"
+		(shape output)
 		(at 170.18 73.66 0)
 		(effects
 			(font
+				(size 1.27 1.27)
+			)
+			(justify left)
+		)
+	)
+	(hierarchical_label "Green_LED"
+		(shape output)
+		(at 114.3 104.14 180)
+		(effects
+			(font
+				(size 1.27 1.27)
+			)
+			(justify right)
+		)
+	)
+	(hierarchical_label "I2S_DIN"
+		(shape output)
+		(at 170.18 63.5 0)
+		(effects
+			(font

Commit message: Single-pager KiCAD
Connections:
- net I2C_SCL: now also U2.41 (19_A5_SCL); no longer U2.37 (15_A1_RX3_SPDIF_IN)
- net I2C_SDA: now also U2.40 (18_A4_SDA); no longer U2.36 (14_A0_TX3_SPDIF_OUT)
- net RST1: now also U2.37 (15_A1_RX3_SPDIF_IN); no longer U2.41 (19_A5_SCL)
- net RST2: now also U2.36 (14_A0_TX3_SPDIF_OUT); no longer U2.40 (18_A4_SDA)
- net I2S2_DIN: now reaches U2.4 (2_OUT2)
- net I2S2_LRC: now reaches U2.5 (3_LRCLK2)
- net I2S2_BCLK: now reaches U2.6 (4_BCLK2)
- net I2S_BCLK renamed I2S1_BCLK
- net I2S_DIN renamed I2S1_DIN
- net I2S_LRC renamed I2S1_LRC
- net UART_RX: no longer names the net of U2.2 (0_RX1_CRX2_CS1)
- net UART_TX: no longer names the net of U2.3 (1_TX1_CTX2_MISO1)
- no-connect marks 41 -> 40
Changed lines of the file:
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@@
-	)
-	(no_connect
-		(at 114.3 66.04)
-	)
-	(no_connect
-		(at 114.3 63.5)
 	)
 	(no_connect
@@
 	)
 	(no_connect
+		(at 114.3 55.88)
+	)
+	(no_connect
 		(at 138.43 140.97)
 	)
@@
 	)
 	(no_connect
+		(at 114.3 58.42)
+	)
+	(no_connect
 		(at 114.3 91.44)
 	)
@@
 	(no_connect
 		(at 170.18 128.27)
-	)
-	(no_connect
-		(at 114.3 60.96)
 	)
 	(no_connect
@@
 	(wire
 		(pts
-			(xy 172.72 88.9) (xy 170.18 88.9)
+			(xy 173.99 88.9) (xy 170.18 88.9)
 		)
 		(stroke
@@
 		)
 	)
+	(hierarchical_label "I2S2_DIN"
+		(shape output)
+		(at 114.3 60.96 180)
+		(effects
+			(font
+				(size 1.27 1.27)
+			)
+			(justify right)
+		)
+	)
 	(hierarchical_label "Red_Button"
 		(shape output)
@@
 		)
 	)
-	(hierarchical_label "I2S_BCLK"
+	(hierarchical_label "I2S1_BCLK"
 		(shape output)
 		(at 170.18 66.04 0)
@@
 		)
 	)
-	(hierarchical_label "I2S_LRC"
+	(hierarchical_label "I2S1_LRC"
 		(shape output)
 		(at 170.18 68.58 0)
@@
 		)
 	)
-	(hierarchical_label "RST1"
+	(hierarchical_label "SPI_CS2"
+		(shape output)
+		(at 170.18 78.74 0)
+		(effects
+			(font
+				(size 1.27 1.27)
+			)
+			(justify left)
+		)
+	)
+	(hierarchical_label "SPI_SDI"
+		(shape output)
+		(at 114.3 83.82 180)
+		(effects
+			(font
+				(size 1.27 1.27)
+			)
+			(justify right)
+		)
+	)
+	(hierarchical_label "SPI_SCK"
+		(shape output)
+		(at 170.18 86.36 0)
+		(effects
+			(font
+				(size 1.27 1.27)
+			)
+			(justify left)
+		)
+	)
+	(hierarchical_label "I2C_SCL"
 		(shape output)
 		(at 170.18 71.12 0)
@@
 		)
 	)
-	(hierarchical_label "SPI_CS2"
-		(shape output)
-		(at 170.18 78.74 0)
-		(effects
-			(font
-				(size 1.27 1.27)
-			)
-			(justify left)
-		)
-	)
-	(hierarchical_label "SPI_SDI"
-		(shape output)
-		(at 114.3 83.82 180)
-		(effects
-			(font
-				(size 1.27 1.27)
-			)
-			(justify right)
-		)
-	)
-	(hierarchical_label "SPI_SCK"
-		(shape output)
-		(at 170.18 86.36 0)
-		(effects
-			(font
-				(size 1.27 1.27)
-			)
-			(justify left)
-		)
-	)
-	(hierarchical_label "UART_RX"
-		(shape input)
-		(at 114.3 55.88 180)
-		(effects
-			(font
-				(size 1.27 1.27)
-			)
-			(justify right)
-		)
-	)
-	(hierarchical_label "UART_TX"
-		(shape output)
-		(at 114.3 58.42 180)
-		(effects
-			(font
-				(size 1.27 1.27)
-			)
-			(justify right)
-		)
-	)
 	(hierarchical_label "Green_Button"
 		(shape output)
@@
 		)
 	)
-	(hierarchical_label "I2C_SCL"
-		(shape output)
-		(at 170.18 81.28 0)
-		(effects
-			(font
-				(size 1.27 1.27)
-			)
-			(justify left)
-		)
-	)
 	(hierarchical_label "Red_LED"
 		(shape output)
@@
 			)
 			(justify right)
+		)
+	)
+	(hierarchical_label "RST2"
+		(shape output)
+		(at 170.18 83.82 0)
+		(effects
+			(font
+				(size 1.27 1.27)
+			)
+			(justify left)
 		)
 	)
@@
 		)
 	)
+	(hierarchical_label "White_Button"
+		(shape output)
+		(at 114.3 93.98 180)
+		(effects
+			(font
+				(size 1.27 1.27)
+			)
+			(justify right)
+		)
+	)
+	(hierarchical_label "Green_LED"
+		(shape output)
+		(at 114.3 104.14 180)
+		(effects
+			(font
+				(size 1.27 1.27)
+			)
+			(justify right)
+		)
+	)
+	(hierarchical_label "I2S1_DIN"
+		(shape output)
+		(at 170.18 63.5 0)
+		(effects
+			(font
+				(size 1.27 1.27)
+			)
+			(justify left)
+		)
+	)
+	(hierarchical_label "I2S2_LRC"
+		(shape output)
+		(at 114.3 63.5 180)
+		(effects
+			(font
+				(size 1.27 1.27)
+			)
+			(justify right)
+		)
+	)
+	(hierarchical_label "SPI_CS"
+		(shape output)
+		(at 114.3 81.28 180)
+		(effects
+			(font
+				(size 1.27 1.27)
+			)
+			(justify right)
+		)
+	)
+	(hierarchical_label "RST1"
+		(shape output)
+		(at 170.18 81.28 0)
+		(effects
+			(font
+				(size 1.27 1.27)
+			)
+			(justify left)
+		)
+	)
 	(hierarchical_label "I2C_SDA"
 		(shape bidirectional)
-		(at 170.18 83.82 0)
-		(effects
-			(font
-				(size 1.27 1.27)
-			)
-			(justify left)
-		)
-	)
-	(hierarchical_label "White_Button"
-		(shape output)
-		(at 114.3 93.98 180)
-		(effects
-			(font
-				(size 1.27 1.27)
-			)
-			(justify right)
-		)
-	)
-	(hierarchical_label "RST2"
-		(shape output)
 		(at 170.18 73.66 0)
 		(effects
@@
 		)
 	)
-	(hierarchical_label "Green_LED"
-		(shape output)
-		(at 114.3 104.14 180)
-		(effects
-			(font
-				(size 1.27 1.27)
-			)
-			(justify right)
-		)
-	)
-	(hierarchical_label "I2S_DIN"
-		(shape output)
-		(at 170.18 63.5 0)
-		(effects
-			(font
-				(size 1.27 1.27)
-			)
-			(justify left)
-		)
-	)
-	(hierarchical_label "SPI_CS"
-		(shape output)
-		(at 114.3 81.28 180)
+	(hierarchical_label "I2S2_BCLK"
+		(shape output)
+		(at 114.3 66.04 180)
 		(effects
 			(font
@@
 	(symbol
 		(lib_id "power:GND")
-		(at 172.72 88.9 0)
+		(at 173.99 88.9 0)
 		(unit 1)
 		(exclude_from_sim no)
@@
 		(fields_autoplaced yes)
 		(property "Reference" "#PWR025"
-			(at 172.72 95.25 0)
+			(at 173.99 95.25 0)
 			(effects
 				(font
@@
 		)
 		(property "Value" "GND"
-			(at 172.72 93.98 0)
+			(at 173.99 93.98 0)
 			(effects
 				(font
@@
 		)
 		(property "Footprint" ""
-			(at 172.72 88.9 0)
+			(at 173.99 88.9 0)
 			(effects
 				(font
@@
 		)
 		(property "Datasheet" ""
-			(at 172.72 88.9 0)
+			(at 173.99 88.9 0)
 			(effects
 				(font
@@
 		)
 		(property "Description" "Power symbol creates a global label with name \"GND\" , ground"
-			(at 172.72 88.9 0)
-			(effects
-				(font
+			(at 173.99 88.9 0)
+			(effects
+				(font

Commit message: force sensor oobs
Connections:
- net I2S1_DIN: now also U2.9 (7_RX2_OUT1A); no longer U2.44 (22_A8_CTX1)
- new net FORCE_IN: U2.44 (22_A8_CTX1)
- no-connect marks 40 -> 39
Changed lines of the file:
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@@
-	)
-	(no_connect
-		(at 114.3 73.66)
 	)
 	(no_connect
@@
 		)
 	)
+	(hierarchical_label "FORCE_IN"
+		(shape input)
+		(at 170.18 63.5 0)
+		(effects
+			(font
+				(size 1.27 1.27)
+			)
+			(justify left)
+		)
+	)
 	(hierarchical_label "I2S1_LRC"
 		(shape output)
@@
 	(hierarchical_label "I2S1_DIN"
 		(shape output)
-		(at 170.18 63.5 0)
-		(effects
-			(font
-				(size 1.27 1.27)
-			)
-			(justify left)
-		)
-	)
+		(at 114.3 73.66 180)
+		(effects
+			(font
+				(size 1.27 1.27)
+			)
+			(justify right)
+		)
+	)

Commit message: I2S Combination and Screen driver fixes
Connections:
- net I2S1_BCLK renamed I2S_BCLK
- net I2S1_DIN renamed I2S_DIN
- net I2S1_LRC renamed I2S_LRC
- net I2S2_BCLK: no longer names the net of U2.6 (4_BCLK2)
- net I2S2_DIN: no longer names the net of U2.4 (2_OUT2)
- net I2S2_LRC: no longer names the net of U2.5 (3_LRCLK2)
- no-connect marks 39 -> 42
Changed lines of the file:
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@@
+	)
+	(no_connect
+		(at 114.3 60.96)
 	)
 	(no_connect
@@
 	)
 	(no_connect
+		(at 114.3 63.5)
+	)
+	(no_connect
 		(at 170.18 49.53)
 	)
@@
 	(no_connect
 		(at 170.18 130.81)
+	)
+	(no_connect
+		(at 114.3 66.04)
 	)
 	(wire
@@
 		)
 	)
-	(hierarchical_label "I2S2_DIN"
-		(shape output)
-		(at 114.3 60.96 180)
-		(effects
-			(font
-				(size 1.27 1.27)
-			)
-			(justify right)
-		)
-	)
 	(hierarchical_label "Red_Button"
 		(shape output)
@@
 		)
 	)
-	(hierarchical_label "I2S1_BCLK"
+	(hierarchical_label "I2S_BCLK"
 		(shape output)
 		(at 170.18 66.04 0)
@@
 		)
 	)
-	(hierarchical_label "I2S1_LRC"
+	(hierarchical_label "I2S_LRC"
 		(shape output)
 		(at 170.18 68.58 0)
@@
 		)
 	)
-	(hierarchical_label "I2S1_DIN"
+	(hierarchical_label "I2S_DIN"
 		(shape output)
 		(at 114.3 73.66 180)
-		(effects
-			(font
-				(size 1.27 1.27)
-			)
-			(justify right)
-		)
-	)
-	(hierarchical_label "I2S2_LRC"
-		(shape output)
-		(at 114.3 63.5 180)
 		(effects
 			(font
@@
 		)
 	)
-	(hierarchical_label "I2S2_BCLK"
-		(shape output)
-		(at 114.3 66.04 180)
-		(effects
-			(font
-				(size 1.27 1.27)
-			)
-			(justify right)
-		)
-	)
