File: M6/CPR Machine Schematic/Microcontroller.kicad_sch (KiCad schematic)
At the start: 1 part, among them U2 Teensy4.1

Commit message: more kicad
Connections:
- net RST2 is gone; now on net Red_Button: U2.36 (14_A0_TX3_SPDIF_OUT)
- net SPI_CS3 is gone; now on net SPI_CS2: U2.39 (17_A3_TX4_SDA1)
- net Red_Button: no longer U2.18 (26_A12_MOSI1)
- net Red_LED: now also U2.38 (16_A2_RX4_SCL1); no longer U2.19 (27_A13_SCK1)
- net SPI_CS2: no longer U2.38 (16_A2_RX4_SCL1)
- net SPI1_MISO: now reaches U2.3 (1_TX1_CTX2_MISO1)
- net SPI_CS renamed SPI_CS1
- net SPI_INT renamed SPI_INT1
- new net SPI1_MOSI: U2.18 (26_A12_MOSI1)
- new net SPI1_SCK: U2.19 (27_A13_SCK1)
- no-connect marks 42 -> 39
Changed lines of the file:
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@@
 	(paper "A4")
 	(no_connect
-		(at 114.3 106.68)
-	)
-	(no_connect
 		(at 142.24 140.97)
 	)
@@
 	)
 	(no_connect
-		(at 114.3 109.22)
-	)
-	(no_connect
 		(at 114.3 128.27)
 	)
@@
 	(no_connect
 		(at 170.18 123.19)
-	)
-	(no_connect
-		(at 114.3 58.42)
 	)
 	(no_connect
@@
 		)
 	)
-	(hierarchical_label "SPI_CS3"
-		(shape output)
-		(at 170.18 76.2 0)
-		(effects
-			(font
-				(size 1.27 1.27)
-			)
-			(justify left)
-		)
-	)
 	(hierarchical_label "SPI_SDO"
 		(shape input)
@@
 	(hierarchical_label "Red_Button"
 		(shape output)
-		(at 114.3 96.52 180)
-		(effects
-			(font
-				(size 1.27 1.27)
-			)
-			(justify right)
+		(at 170.18 83.82 0)
+		(effects
+			(font
+				(size 1.27 1.27)
+			)
+			(justify left)
 		)
 	)
@@
 	(hierarchical_label "SPI_CS2"
 		(shape output)
+		(at 170.18 76.2 0)
+		(effects
+			(font
+				(size 1.27 1.27)
+			)
+			(justify left)
+		)
+	)
+	(hierarchical_label "SPI_SDI"
+		(shape output)
+		(at 114.3 83.82 180)
+		(effects
+			(font
+				(size 1.27 1.27)
+			)
+			(justify right)
+		)
+	)
+	(hierarchical_label "SPI_SCK"
+		(shape output)
+		(at 170.18 86.36 0)
+		(effects
+			(font
+				(size 1.27 1.27)
+			)
+			(justify left)
+		)
+	)
+	(hierarchical_label "SPI1_MISO"
+		(shape input)
+		(at 114.3 58.42 180)
+		(effects
+			(font
+				(size 1.27 1.27)
+			)
+			(justify right)
+		)
+	)
+	(hierarchical_label "I2C_SCL"
+		(shape output)
+		(at 170.18 71.12 0)
+		(effects
+			(font
+				(size 1.27 1.27)
+			)
+			(justify left)
+		)
+	)
+	(hierarchical_label "Green_Button"
+		(shape output)
+		(at 114.3 101.6 180)
+		(effects
+			(font
+				(size 1.27 1.27)
+			)
+			(justify right)
+		)
+	)
+	(hierarchical_label "SPI1_SCK"
+		(shape output)
+		(at 114.3 99.06 180)
+		(effects
+			(font
+				(size 1.27 1.27)
+			)
+			(justify right)
+		)
+	)
+	(hierarchical_label "Red_LED"
+		(shape output)
 		(at 170.18 78.74 0)
 		(effects
@@
 		)
 	)
-	(hierarchical_label "SPI_SDI"
-		(shape output)
-		(at 114.3 83.82 180)
-		(effects
-			(font
-				(size 1.27 1.27)
-			)
-			(justify right)
-		)
-	)
-	(hierarchical_label "SPI_SCK"
-		(shape output)
-		(at 170.18 86.36 0)
-		(effects
-			(font
-				(size 1.27 1.27)
-			)
-			(justify left)
-		)
-	)
-	(hierarchical_label "I2C_SCL"
-		(shape output)
-		(at 170.18 71.12 0)
-		(effects
-			(font
-				(size 1.27 1.27)
-			)
-			(justify left)
-		)
-	)
-	(hierarchical_label "Green_Button"
-		(shape output)
-		(at 114.3 101.6 180)
-		(effects
-			(font
-				(size 1.27 1.27)
-			)
-			(justify right)
-		)
-	)
-	(hierarchical_label "Red_LED"
-		(shape output)
-		(at 114.3 99.06 180)
-		(effects
-			(font
-				(size 1.27 1.27)
-			)
-			(justify right)
-		)
-	)
-	(hierarchical_label "RST2"
-		(shape output)
-		(at 170.18 83.82 0)
-		(effects
-			(font
-				(size 1.27 1.27)
-			)
-			(justify left)
-		)
-	)
-	(hierarchical_label "SPI_INT"
+	(hierarchical_label "SPI_INT1"
 		(shape input)
 		(at 114.3 78.74 180)
@@
 		)
 	)
+	(hierarchical_label "SPI1_MOSI"
+		(shape output)
+		(at 114.3 96.52 180)
+		(effects
+			(font
+				(size 1.27 1.27)
+			)
+			(justify right)
+		)
+	)
 	(hierarchical_label "Green_LED"
 		(shape output)
@@
 		)
 	)
-	(hierarchical_label "SPI_CS"
+	(hierarchical_label "SPI_CS1"
 		(shape output)
 		(at 114.3 81.28 180)
