File: M6/CPR Machine Schematic/CPR Machine Schematic.kicad_sch (KiCad schematic)
At the start: 0 parts

Commit message: more kicad
Other:
- sheet HMI_No_Raspi ports: added none; removed RST2, SPI_CS3
- sheet Microcontroller ports: added SPI1_MISO, SPI1_MOSI, SPI1_SCK, SPI_CS1, SPI_INT1; removed RST2, SPI_CS, SPI_CS3, SPI_INT
Changed lines of the file:
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@@
 	(generator_version "9.0")
 	(paper "A4")
-	(junction
-		(at 121.92 85.09)
-		(diameter 0)
-		(color 0 0 0 0)
-	)
-	(junction
-		(at 118.11 81.28)
-		(diameter 0)
-		(color 0 0 0 0)
-	)
-	(junction
-		(at 114.3 77.47)
-		(diameter 0)
-		(color 0 0 0 0)
+	(wire
+		(pts
+			(xy 110.49 81.28) (xy 134.62 81.28)
+		)
+		(stroke
+			(width 0)
+			(type default)
+		)
 	)
 	(wire
@@
 	(wire
 		(pts
-			(xy 193.04 73.66) (xy 187.96 73.66)
-		)
-		(stroke
-			(width 0)
-			(type default)
-		)
-	)
-	(wire
-		(pts
-			(xy 180.34 81.28) (xy 180.34 64.77)
-		)
-		(stroke
-			(width 0)
-			(type default)
-		)
-	)
-	(wire
-		(pts
-			(xy 180.34 64.77) (xy 121.92 64.77)
+			(xy 110.49 85.09) (xy 134.62 85.09)
 		)
 		(stroke
@@
 	(wire
 		(pts
-			(xy 173.99 92.71) (xy 193.04 92.71)
-		)
-		(stroke
-			(width 0)
-			(type default)
-		)
-	)
-	(wire
-		(pts
 			(xy 173.99 123.19) (xy 193.04 123.19)
 		)
@@
 	(wire
 		(pts
-			(xy 110.49 81.28) (xy 118.11 81.28)
-		)
-		(stroke
-			(width 0)
-			(type default)
-		)
-	)
-	(wire
-		(pts
 			(xy 110.49 121.92) (xy 134.62 121.92)
 		)
@@
 	(wire
 		(pts
-			(xy 118.11 81.28) (xy 134.62 81.28)
-		)
-		(stroke
-			(width 0)
-			(type default)
-		)
-	)
-	(wire
-		(pts
 			(xy 173.99 118.11) (xy 193.04 118.11)
 		)
@@
 	(wire
 		(pts
-			(xy 110.49 77.47) (xy 114.3 77.47)
-		)
-		(stroke
-			(width 0)
-			(type default)
-		)
-	)
-	(wire
-		(pts
-			(xy 187.96 57.15) (xy 114.3 57.15)
-		)
-		(stroke
-			(width 0)
-			(type default)
-		)
-	)
-	(wire
-		(pts
-			(xy 193.04 77.47) (xy 184.15 77.47)
+			(xy 173.99 73.66) (xy 193.04 73.66)
 		)
 		(stroke
@@
 	(wire
 		(pts
-			(xy 121.92 64.77) (xy 121.92 85.09)
-		)
-		(stroke
-			(width 0)
-			(type default)
-		)
-	)
-	(wire
-		(pts
 			(xy 173.99 85.09) (xy 193.04 85.09)
 		)
@@
 	(wire
 		(pts
-			(xy 118.11 60.96) (xy 118.11 81.28)
-		)
-		(stroke
-			(width 0)
-			(type default)
-		)
-	)
-	(wire
-		(pts
-			(xy 114.3 57.15) (xy 114.3 77.47)
-		)
-		(stroke
-			(width 0)
-			(type default)
-		)
-	)
-	(wire
-		(pts
-			(xy 184.15 60.96) (xy 118.11 60.96)
-		)
-		(stroke
-			(width 0)
-			(type default)
-		)
-	)
-	(wire
-		(pts
-			(xy 193.04 81.28) (xy 180.34 81.28)
-		)
-		(stroke
-			(width 0)
-			(type default)
-		)
-	)
-	(wire
-		(pts
-			(xy 173.99 96.52) (xy 193.04 96.52)
+			(xy 173.99 81.28) (xy 193.04 81.28)
 		)
 		(stroke
@@
 	(wire
 		(pts
+			(xy 110.49 77.47) (xy 134.62 77.47)
+		)
+		(stroke
+			(width 0)
+			(type default)
+		)
+	)
+	(wire
+		(pts
 			(xy 173.99 120.65) (xy 193.04 120.65)
 		)
@@
 	(wire
 		(pts
-			(xy 114.3 77.47) (xy 134.62 77.47)
-		)
-		(stroke
-			(width 0)
-			(type default)
-		)
-	)
-	(wire
-		(pts
 			(xy 110.49 92.71) (xy 134.62 92.71)
 		)
@@
 	(wire
 		(pts
-			(xy 110.49 85.09) (xy 121.92 85.09)
-		)
-		(stroke
-			(width 0)
-			(type default)
-		)
-	)
-	(wire
-		(pts
-			(xy 187.96 73.66) (xy 187.96 57.15)
-		)
-		(stroke
-			(width 0)
-			(type default)
-		)
-	)
-	(wire
-		(pts
-			(xy 184.15 77.47) (xy 184.15 60.96)
-		)
-		(stroke
-			(width 0)
-			(type default)
-		)
-	)
-	(wire
-		(pts
-			(xy 121.92 85.09) (xy 134.62 85.09)
-		)
-		(stroke
-			(width 0)
-			(type default)
-		)
-	)
-	(wire
-		(pts
 			(xy 173.99 105.41) (xy 193.04 105.41)
+		)
+		(stroke
+			(width 0)
+			(type default)
+		)
+	)
+	(wire
+		(pts
+			(xy 173.99 77.47) (xy 193.04 77.47)
 		)
 		(stroke
@@
 		)
 		(pin "RST1" input
-			(at 193.04 92.71 180)
-			(effects
-				(font
-					(size 1.27 1.27)
-				)
-				(justify left)
-			)
-		)
-		(pin "RST2" input
-			(at 193.04 96.52 180)
+			(at 193.04 88.9 180)
 			(effects
 				(font
@@
 		(pin "White_Button" input
 			(at 193.04 118.11 180)
-			(effects
-				(font
-					(size 1.27 1.27)
-				)
-				(justify left)
-			)
-		)
-		(pin "SPI_CS3" input
-			(at 193.04 88.9 180)
 			(effects
 				(font
@@
 			)
 		)
-		(pin "SPI_INT" input
+		(pin "SPI_INT1" input
 			(at 134.62 92.71 180)
 			(effects
@@
 			)
 		)
-		(pin "SPI_CS" output
+		(pin "SPI_CS1" output
 			(at 134.62 88.9 180)
 			(effects
@@
 		)
 		(pin "SPI_SDI" output
-			(at 134.62 81.28 180)
-			(effects
-				(font
-					(size 1.27 1.27)
-				)
-				(justify left)
+			(at 173.99 77.47 0)
+			(effects
+				(font
+					(size 1.27 1.27)
+				)
+				(justify right)
 			)
 		)
 		(pin "SPI_SDO" input
-			(at 134.62 85.09 180)
-			(effects
-				(font
-					(size 1.27 1.27)
-				)
-				(justify left)
+			(at 173.99 81.28 0)
+			(effects
+				(font
+					(size 1.27 1.27)
+				)
+				(justify right)
 			)
 		)
 		(pin "SPI_SCK" output
-			(at 134.62 77.47 180)
-			(effects
-				(font
-					(size 1.27 1.27)
-				)
-				(justify left)
+			(at 173.99 73.66 0)
+			(effects
+				(font
+					(size 1.27 1.27)
+				)
+				(justify right)
 			)
 		)
@@
 			)
 		)
-		(pin "SPI_CS3" output
+		(pin "RST1" output
 			(at 173.99 88.9 0)
-			(effects
-				(font
-					(size 1.27 1.27)
-				)
-				(justify right)
-			)
-		)
-		(pin "RST1" output
-			(at 173.99 92.71 0)
-			(effects
-				(font
-					(size 1.27 1.27)
-				)
-				(justify right)
-			)
-		)
-		(pin "RST2" output
-			(at 173.99 96.52 0)
 			(effects
 				(font
@@
 			)
 		)
+		(pin "SPI1_MOSI" output
+			(at 134.62 81.28 180)
+			(effects
+				(font
+					(size 1.27 1.27)
+				)
+				(justify left)
+			)
+		)
+		(pin "SPI1_SCK" output
+			(at 134.62 77.47 180)
+			(effects
+				(font
+					(size 1.27 1.27)
+				)
+				(justify left)
+			)
+		)
+		(pin "SPI1_MISO" input
+			(at 134.62 85.09 180)
+			(effects
+				(font
+					(size 1.27 1.27)
+				)
+				(justify left)
+			)
+		)

Commit message: Start of Schematic V2
Other:
- removed sheet HMI_No_Raspi
- removed sheet Microcontroller
- removed sheet Motor Control
- added sheet HMI_Raspi (HMI_Raspi.kicad_sch)
- added sheet Raspi (Raspi.kicad_sch)

Commit message: More PCB Progress
All Footprints
Other:
- sheet HMI_Raspi ports: added Laser_PWM; removed White_Button
- sheet Raspi ports: added Laser_PWM; removed White_Button
- sheet Sensing ports: added FORCE_IN; removed FORCE_PIN
Changed lines of the file:
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@@
+	(wire
+		(pts
+			(xy 166.37 86.36) (xy 176.53 86.36)
+		)
+		(stroke
+			(width 0)
+			(type default)
+		)
+	)
 	(wire
 		(pts
@@
 		(pts
 			(xy 166.37 78.74) (xy 176.53 78.74)
-		)
-		(stroke
-			(width 0)
-			(type default)
-		)
-	)
-	(wire
-		(pts
-			(xy 166.37 86.36) (xy 176.53 86.36)
 		)
 		(stroke
@@
 			)
 		)
-		(pin "FORCE_PIN" output
+		(pin "FORCE_IN" output
 			(at 110.49 85.09 0)
 			(effects
@@
 			)
 		)
-		(pin "White_Button" input
-			(at 176.53 86.36 180)
-			(effects
-				(font
-					(size 1.27 1.27)
-				)
-				(justify left)
-			)
-		)
 		(pin "Stop_Enable" input
 			(at 176.53 83.82 180)
@@
 		(pin "Go_Enable" input
 			(at 176.53 78.74 180)
+			(effects
+				(font
+					(size 1.27 1.27)
+				)
+				(justify left)
+			)
+		)
+		(pin "Laser_PWM" input
+			(at 176.53 86.36 180)
 			(effects
 				(font
@@
 			)
 		)
-		(pin "White_Button" output
-			(at 166.37 86.36 0)
-			(effects
-				(font
-					(size 1.27 1.27)
-				)
-				(justify right)
-			)
-		)
 		(pin "Stop_Enable" output
 			(at 166.37 83.82 0)
@@
 			(effects
 				(font
+					(size 1.27 1.27)
+				)
+				(justify right)
+			)
+		)
+		(pin "Laser_PWM" output
+			(at 166.37 86.36 0)
+			(effects
+				(font

Commit message: PCB Feedback V1
Other:
- sheet Raspi ports: added none; removed FORCE_IN
- sheet Sensing ports: added none; removed FORCE_IN
Changed lines of the file:
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@@
-	(wire
-		(pts
-			(xy 110.49 85.09) (xy 120.65 85.09)
-		)
-		(stroke
-			(width 0)
-			(type default)
-		)
-	)
 	(wire
 		(pts
@@
 	(wire
 		(pts
-			(xy 110.49 77.47) (xy 120.65 77.47)
+			(xy 110.49 80.01) (xy 120.65 80.01)
 		)
 		(stroke
@@
 	(wire
 		(pts
-			(xy 110.49 81.28) (xy 120.65 81.28)
+			(xy 110.49 83.82) (xy 120.65 83.82)
 		)
 		(stroke
@@
 		)
 		(pin "I2C_SCL" input
-			(at 110.49 77.47 0)
+			(at 110.49 80.01 0)
 			(effects
 				(font
@@
 		)
 		(pin "I2C_SDA" bidirectional
-			(at 110.49 81.28 0)
-			(effects
-				(font
-					(size 1.27 1.27)
-				)
-				(justify right)
-			)
-		)
-		(pin "FORCE_IN" output
-			(at 110.49 85.09 0)
+			(at 110.49 83.82 0)
 			(effects
 				(font
@@
 			)
 		)
-		(pin "FORCE_IN" input
-			(at 120.65 85.09 180)
-			(effects
-				(font
-					(size 1.27 1.27)
-				)
-				(justify left)
-			)
-		)
 		(pin "I2C_SDA" bidirectional
-			(at 120.65 81.28 180)
+			(at 120.65 83.82 180)
 			(effects
 				(font
@@
 		)
 		(pin "I2C_SCL" bidirectional
-			(at 120.65 77.47 180)
-			(effects
-				(font
+			(at 120.65 80.01 180)
+			(effects
+				(font
