File: M6/CPR Machine Schematic/Raspi.kicad_sch (KiCad schematic)
At the start: 3 parts, among them J13 Raspberry_Pi_2_3, J15 Conn_02x20_Odd_Even

Commit message: Updated ADC Logic Level, Redone Layout, Geographic Reannotation
Parts:
- renumbered J13 to J14, J15 to J8
Connections:
- net MUX Select is gone; now on net GPIO19: J14.35 (GPIO19/MISO1)
Other:
- note added: "3V3 disconnected because of seperate 3V3 source on hat"
Changed lines of the file:
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@@
+		)
+	)
+	(text "3V3 disconnected because of seperate 3V3 source on hat"
+		(exclude_from_sim no)
+		(at 173.228 72.136 0)
+		(effects
+			(font
+				(size 1.27 1.27)
+			)
 		)
 	)
@@
 		)
 	)
+	(label "GPIO19"
+		(at 120.65 105.41 180)
+		(effects
+			(font
+				(size 1.27 1.27)
+			)
+			(justify right bottom)
+		)
+	)
 	(label "GPIO11"
 		(at 161.29 123.19 0)
@@
 		(shape output)
 		(at 120.65 125.73 180)
-		(effects
-			(font
-				(size 1.27 1.27)
-			)
-			(justify right)
-		)
-	)
-	(hierarchical_label "MUX Select"
-		(shape output)
-		(at 120.65 105.41 180)
 		(effects
 			(font
@@
 		(dnp no)
 		(fields_autoplaced yes)
-		(property "Reference" "J13"
+		(property "Reference" "J14"
 			(at 148.1933 74.93 0)
 			(effects
@@
 			(project ""
 				(path "/8991fc77-975f-4978-a089-6b2a5e33f59b/7b515552-6db1-403d-b6a0-a1579d4772aa"
-					(reference "J13")
+					(reference "J14")
 					(unit 1)
 				)
@@
 		(dnp no)
 		(fields_autoplaced yes)
-		(property "Reference" "J15"
+		(property "Reference" "J8"
 			(at 204.47 80.01 0)
 			(effects
@@
 			(project ""
 				(path "/8991fc77-975f-4978-a089-6b2a5e33f59b/7b515552-6db1-403d-b6a0-a1579d4772aa"
-					(reference "J15")
+					(reference "J8")
 					(unit 1)
 				)
