File: M6/CPR Machine Schematic/Sensing.kicad_sch (KiCad schematic)
At the start: 6 parts, among them J12 I2C Port, J8 Force Sensor, U3 MCP6001R

Commit message: PCB Feedback V1
Parts:
- added R17: 90 kOhm, Resistor_SMD:R_1206_3216Metric, symbol Device:R_US
- added R18: 10 kOhm, Resistor_SMD:R_1206_3216Metric, symbol Device:R_US
- added U5: MCP3021A0T-E_OT, 2679:IC_MCP3021A0T-E_OT, symbol Custom_Parts:MCP3021A0T-E_OT
- R16: value 10 kOhm -> 80 Ohm
- U3: value MCP6001R -> MCP6004; footprint Package_TO_SOT_SMD:SOT-23-5 -> MCP6004:SOIC14_SL_MCH
Connections:
- net +5V: now also U3.4 (V+), R17.1, U5.1 (VDD); no longer U3.2 (V+)
- net GND: now also U3.11 (V-), R18.2, U5.2 (VSS); no longer U3.3 (+), U3.5 (V-)
- net I2C_SCL: now also U5.5 (SCL)
- net I2C_SDA: now also U5.4 (SDA)
- net at C13.1, J8.1 (Pin_1), R16.2: now also U3.2 (-); no longer U3.4 (-)
- net FORCE_IN: no longer names the net of C13.2, C_OPT1.2, R16.1, U3.1
- net FORCE_IN: now also U5.3 (AIN)
- new net Vref: R17.2, R18.1, U3.3 (+)
Other:
- moved on the sheet: J8

Commit message: PCB V2 Part 2
Parts:
- C13, C_OPT1: footprint Capacitor_SMD:C_1206_3216Metric -> Capacitor_SMD:C_1206_3216Metric_Pad1.33x1.80mm_HandSolder; digikey (none) -> 1292-1206N470J102CT-ND
- J12: now left out of the parts list
- J8: digikey (none) -> 277-1667-ND
- R16: value 80 Ohm -> 80.6 Ohm; footprint Resistor_SMD:R_1206_3216Metric -> Resistor_SMD:R_1206_3216Metric_Pad1.30x1.75mm_HandSolder; digikey (none) -> 311-80.6FRCT-ND
- R17: footprint Resistor_SMD:R_1206_3216Metric -> Resistor_SMD:R_1206_3216Metric_Pad1.30x1.75mm_HandSolder; digikey (none) -> 13-RT1206DRE0790KLCT-ND
- R18: footprint Resistor_SMD:R_1206_3216Metric -> Resistor_SMD:R_1206_3216Metric_Pad1.30x1.75mm_HandSolder; now left out of the parts list
- U3: digikey (none) -> MCP6004T-I/SLCT-ND
- U5: digikey (none) -> MCP3021A0T-E/OTCT-ND
Changed lines of the file:
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@@
 			)
 		)
-		(property "Footprint" "Capacitor_SMD:C_1206_3216Metric"
+		(property "Footprint" "Capacitor_SMD:C_1206_3216Metric_Pad1.33x1.80mm_HandSolder"
 			(at 73.9648 50.8 0)
 			(effects
@@
 			)
 		)
-		(property "Datasheet" "~"
+		(property "Datasheet" "http://www.passivecomponent.com/wp-content/uploads/datasheet/WTC_MLCC_Middle_and_High_Voltage.pdf"
 			(at 74.93 54.61 0)
 			(effects
@@
 		)
 		(property "Description" "Unpolarized capacitor"
+			(at 74.93 54.61 0)
+			(effects
+				(font
+					(size 1.27 1.27)
+				)
+				(hide yes)
+			)
+		)
+		(property "digikey" "1292-1206N470J102CT-ND"
 			(at 74.93 54.61 0)
 			(effects
@@
 		(unit 1)
 		(exclude_from_sim no)
-		(in_bom yes)
+		(in_bom no)
 		(on_board yes)
 		(dnp no)
@@
 			)
 		)
-		(property "Datasheet" ""
+		(property "Datasheet" "https://ww1.microchip.com/downloads/aemDocuments/documents/APID/ProductDocuments/DataSheets/20001805C.pdf"
 			(at 102.87 48.26 0)
 			(effects
@@
 				)
 				(justify bottom)
+				(hide yes)
+			)
+		)
+		(property "digikey" "MCP3021A0T-E/OTCT-ND"
+			(at 102.87 48.26 0)
+			(effects
+				(font
+					(size 1.27 1.27)
+				)
 				(hide yes)
 			)
@@
 			)
 		)
-		(property "Datasheet" "~"
+		(property "Datasheet" "https://mm.digikey.com/Volume0/opasdata/d220001/medias/docus/909/1935161.pdf"
 			(at 40.64 86.36 0)
 			(effects
@@
 			)
 		)
+		(property "digikey" "277-1667-ND"
+			(at 40.64 86.36 0)
+			(effects
+				(font
+					(size 1.27 1.27)
+				)
+				(hide yes)
+			)
+		)
 		(pin "2"
 		)
@@
 			)
 		)
-		(property "Footprint" "Capacitor_SMD:C_1206_3216Metric"
+		(property "Footprint" "Capacitor_SMD:C_1206_3216Metric_Pad1.33x1.80mm_HandSolder"
 			(at 62.23 79.0448 0)
 			(effects
@@
 			)
 		)
-		(property "Datasheet" "~"
+		(property "Datasheet" "http://www.passivecomponent.com/wp-content/uploads/datasheet/WTC_MLCC_Middle_and_High_Voltage.pdf"
 			(at 58.42 80.01 0)
 			(effects
@@
 			)
 		)
+		(property "digikey" "1292-1206N470J102CT-ND"
+			(at 58.42 80.01 90)
+			(effects
+				(font
+					(size 1.27 1.27)
+				)
+				(hide yes)
+			)
+		)
 		(pin "1"
 		)
@@
 			)
 		)
-		(property "Value" "80 Ohm"
+		(property "Value" "80.6 Ohm"
 			(at 58.42 66.04 90)
 			(effects
@@
 			)
 		)
-		(property "Footprint" "Resistor_SMD:R_1206_3216Metric"
+		(property "Footprint" "Resistor_SMD:R_1206_3216Metric_Pad1.30x1.75mm_HandSolder"
 			(at 58.166 70.866 90)
 			(effects
@@
 			)
 		)
-		(property "Datasheet" "~"
+		(property "Datasheet" "https://yageogroup.com/content/datasheet/asset/file/PYU-RC_GROUP_51_ROHS_L"
 			(at 58.42 69.85 0)
 			(effects
@@
 			)
 		)
+		(property "digikey" "311-80.6FRCT-ND"
+			(at 58.42 69.85 90)
+			(effects
+				(font
+					(size 1.27 1.27)
+				)
+				(hide yes)
+			)
+		)
 		(pin "2"
 		)
@@
 			)
 		)
+		(property "digikey" "MCP6004T-I/SLCT-ND"
+			(at 59.69 48.26 0)
+			(effects
+				(font
+					(size 1.27 1.27)
+				)
+				(hide yes)
+			)
+		)
 		(pin "4"
 		)
@@
 		(unit 1)
 		(exclude_from_sim no)
-		(in_bom yes)
+		(in_bom no)
 		(on_board yes)
 		(dnp no)
@@
 			)
 		)
-		(property "Footprint" "Resistor_SMD:R_1206_3216Metric"
+		(property "Footprint" "Resistor_SMD:R_1206_3216Metric_Pad1.30x1.75mm_HandSolder"
 			(at 35.306 49.784 90)
 			(effects
@@
 			)
 		)
-		(property "Footprint" "Resistor_SMD:R_1206_3216Metric"
+		(property "Footprint" "Resistor_SMD:R_1206_3216Metric_Pad1.30x1.75mm_HandSolder"
 			(at 35.306 42.164 90)
 			(effects
@@
 			)
 		)
-		(property "Datasheet" "~"
+		(property "Datasheet" "https://yageogroup.com/content/datasheet/asset/file/PYU-RT_1-TO-0-01_ROHS_L"
 			(at 34.29 41.91 0)
 			(effects
@@
 			(at 34.29 41.91 0)
 			(effects
+				(font
+					(size 1.27 1.27)
+				)
+				(hide yes)
+			)
+		)
+		(property "digikey" "13-RT1206DRE0790KLCT-ND"
+			(at 34.29 41.91 0)
+			(effects

Commit message: Down with the second buck converter
Parts:
- C_OPT1: now not fitted
Other:
- note added: "Force Sensor Op-Amp & ADC"
- note removed: "Force Sensor & Op-Amps"
Changed lines of the file:
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@@
 		)
 	)
-	(text "Force Sensor & Op-Amps"
+	(text "Force Sensor Op-Amp & ADC"
 		(exclude_from_sim no)
-		(at 33.274 30.226 0)
+		(at 34.29 29.464 0)
 		(effects
 			(font
@@
 		(in_bom yes)
 		(on_board yes)
-		(dnp no)
+		(dnp yes)
 		(fields_autoplaced yes)
 		(property "Reference" "C_OPT1"
