File: M6/CPR Machine Schematic/Sensing.kicad_sch (KiCad schematic)
At the start: 9 parts, among them J12 I2C Port, J8 Force Sensor, U3 MCP6004, U5 MCP3021A0T-E_OT

Commit message: Rewire ADC to run on 3V3 line to match  RPI
Connections:
- net +5V renamed +3V3
Changed lines of the file:
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@@
 			)
 		)
-		(property "Value" "+5V"
-			(at 118.11 38.1 0)
-			(effects
-				(font
-					(size 1.27 1.27)
-				)
+		(property "Value" "+3V3"
+			(at 120.65 41.9099 0)
+			(effects
+				(font
+					(size 1.27 1.27)
+				)
+				(justify left)
 			)
 		)
@@
 			)
 		)
-		(property "Value" "+5V"
-			(at 34.29 33.02 0)
-			(effects
-				(font
-					(size 1.27 1.27)
-				)
+		(property "Value" "+3V3"
+			(at 36.83 36.8299 0)
+			(effects
+				(font
+					(size 1.27 1.27)
+				)
+				(justify left)
 			)
 		)
@@
 			)
 		)
-		(property "Value" "+5V"
-			(at 57.15 35.56 0)
-			(effects
-				(font
-					(size 1.27 1.27)
-				)
-			)
-		)
+		(property "Value" "+3V3"
+			(at 59.69 39.3699 0)
+			(effects
+				(font
+					(size 1.27 1.27)
+				)
+				(justify left)
+			)
+		)
