File: M6/CPR Machine Schematic/Power.kicad_sch (KiCad schematic)
At the start: 65 parts, among them J1 Battery 22.2V IN, J14 Battery, J16 Motor Driver, J2 5V Spare Headers, J3 Power Switch, J4 3V3 Spare Headers, J5 12 Spare headers, J6 Battery Spare headers, J7 GND Spare Headers, Q1 2N3904, Q2 SSM3J332R, Q4 DMMT5401 PNP, Q5 DMMT5401 PNP, Q8 DMG2305UX-EV, SW1 SW_SPST, U1 LT1765EFE-5_PBF, U2 MAX42403AFLB+, U4 12V Buck, U6 3.3V Buck

Commit message: XT30 Connectors to battery instead of screw term
Parts:
- J1, J3: footprint TerminalBlock:TerminalBlock_MaiXu_MX126-5.0-02P_1x02_P5.00mm -> Connector_AMASS:AMASS_XT30PW-M_1x02_P2.50mm_Horizontal
Changed lines of the file:
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@@
 			)
 		)
-		(property "Footprint" "TerminalBlock:TerminalBlock_MaiXu_MX126-5.0-02P_1x02_P5.00mm"
+		(property "Footprint" "Connector_AMASS:AMASS_XT30PW-M_1x02_P2.50mm_Horizontal"
 			(at 24.13 38.1 0)
 			(effects
@@
 			)
 		)
-		(property "Footprint" "TerminalBlock:TerminalBlock_MaiXu_MX126-5.0-02P_1x02_P5.00mm"
+		(property "Footprint" "Connector_AMASS:AMASS_XT30PW-M_1x02_P2.50mm_Horizontal"
 			(at 24.13 20.32 0)
 			(effects

Commit message: Updated ADC Logic Level, Redone Layout, Geographic Reannotation
Parts:
- removed C10: 0.18 uF, Capacitor_SMD:C_1206_3216Metric_Pad1.33x1.80mm_HandSolder, symbol Device:C
- removed C11: 330 pF, Capacitor_SMD:C_1206_3216Metric_Pad1.33x1.80mm_HandSolder, symbol Device:C
- removed C12: 15 nF, Capacitor_SMD:C_1206_3216Metric_Pad1.33x1.80mm_HandSolder, symbol Device:C
- removed C9: 2.2 uF, Capacitor_SMD:C_1206_3216Metric_Pad1.33x1.80mm_HandSolder, symbol Device:C
- removed D2: B220a, Diode_SMD:D_SMA_Handsoldering, symbol Diode:B220
- removed D3: SS24, Diode_SMD:D_SMB_Handsoldering, symbol Diode:SS24
- removed L2: 6.8 uH, SRU8043_6R8Y:IND_BOURNS_SRU8043, symbol Device:L
- removed Q1: 2N3904, Package_TO_SOT_THT:TO-92_Inline_Wide, symbol Transistor_BJT:2N3904
- removed R4: 49.9 kOhm, Resistor_SMD:R_1206_3216Metric_Pad1.30x1.75mm_HandSolder, symbol Device:R_US
- removed R7: 2 kOhm, Resistor_SMD:R_1206_3216Metric_Pad1.30x1.75mm_HandSolder, symbol Device:R_US
- removed R8: 47 kOhm, Resistor_SMD:R_1206_3216Metric_Pad1.30x1.75mm_HandSolder, symbol Device:R_US
- removed U1: LT1765EFE-5_PBF, LT1765EFE_5_PBF:SOP65P640X110-17N, symbol Custom_Parts:LT1765EFE-5_PBF
- J1: digikey 277-1667-ND -> (none); gobilda (none) -> 3803-0033-0002; now in the parts list
- J2: renamed from J3; digikey 277-1667-ND -> (none); gobilda (none) -> 3803-0033-0002; now in the parts list
- renumbered C8 to C1, C1 to C2, C5 to C3, C7 to C4, C3 to C5, H4 to H1, H3 to H2, H1 to H3, J2 to J3, J7 to J4, J4 to J5, J5 to J6, J6 to J7, J14 to J_EXT1, Q4 to Q1, Q8 to Q3, Q5 to Q4, R13 to R1, R25 to R10, R26 to R11, R14 to R2, R9 to R3, R10 to R4, R11 to R5, R2 to R6, R1 to R7, R3 to R8, R12 to R9, TP2 to TP1, TP3 to TP2, TP4 to TP3, TP1 to TP4, U6 to U1, U4 to U2, U2 to U3
Connections:
- net +12V: no longer U1.1 (Vin)
- net +5V: now also U1.1 (Vin)
Other:
- note added: "Placeholder 3V3 Converter"
- note added: "Power Test Points"
- note removed: "12V - 5V Regulator DEPRICATED"
- note removed: "Placeholder 12V-3V Converter"
- note removed: "Test Points"
- moved on the sheet: C1, C2, C3, C4, C5, CIN1, CIN2, COUT1, COUT2, L1, Q3, Q4A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
